Commit message: HW 4

File: assign1/src/firstModel/urdf/myfirst.urdf (robot description, URDF)
Before this commit: robot multipleshapes, 5 links, 4 joints
Links:
- removed link end_effector
- link base_link: mass None -> 100; geometry collision box size=1 1 0.1; visual box size=1 1 0.1
- link link_1: mass None -> 10; geometry collision cylinder length=0.1 radius=0.1; visual cylinder length=0.1 radius=0.1
- link link_2: mass None -> 10; geometry collision cylinder length=0.1 radius=0.1; visual cylinder length=0.1 radius=0.1
- link link_3: mass None -> 10; geometry collision cylinder length=0.1 radius=0.1; visual cylinder length=0.1 radius=0.1
Joints:
- removed joint link_3_to_end_effector
- joint base_to_link_1: origin (none) -> xyz=0 0 0 rpy=0 0 0
- joint link_1_to_link_2: origin xyz=0 0 1 rpy=1.5707963267948966 0 0 -> xyz=0 0 0.6 rpy=1.5707963267948966 0 0
- joint link_2_to_link_3: axis (none) -> 0 0 1; limit (none) -> lower=-0.7853981633974483 upper=3.141592653589793 effort=100 velocity=1.0; origin xyz=1 0 0 rpy=1.5707963267948966 0 1.5707963267948966 -> xyz=0 0.6 0 rpy=0 0 0; type fixed -> revolute

Commit message: modified:   assign1/src/firstModel/urdf/myfirst.urdf

File: assign1/src/firstModel/urdf/myfirst.urdf (robot description, URDF)
Before this commit: robot 3dof_robot, 4 links, 3 joints
Links:
- added link end_effector, mass 10; collision box size=0.4 0.4 0.05; visual box size=0.4 0.4 0.05
- link base_link: geometry visual box size=1 1 0.1
- link link_1: geometry collision cylinder length=0.475 radius=0.2; visual cylinder length=0.475 radius=0.2
- link link_2: geometry collision cylinder length=0.2 radius=0.2; visual cylinder length=0.2 radius=0.2
- link link_3: geometry collision box size=0.4 0.4 0.4; visual box size=0.4 0.4 0.4
Joints:
- added joint link_3_to_end_effector: type prismatic, parent link_3, child end_effector, origin xyz=0 0 0.3 rpy=0 0 0, axis 0 0 1, limit lower=0 upper=0.5 effort=100 velocity=1.0
- joint link_1_to_link_2: limit (none) -> lower=-0.7853981633974483 upper=3.141592653589793 effort=100 velocity=1.0; origin xyz=0 0 0.6 rpy=1.5707963267948966 0 0 -> xyz=0 0 1 rpy=1.5707963267948966 0 0; type continuous -> revolute
- joint link_2_to_link_3: axis 0 0 1 -> (none); limit lower=-0.7853981633974483 upper=3.141592653589793 effort=100 velocity=1.0 -> (none); origin xyz=0 0.6 0 rpy=0 0 0 -> xyz=1 0 0 rpy=1.5707963267948966 0 1.5707963267948966; type revolute -> fixed
